Commit message: [FIX] Updated robot model
Reduced robot size.

File: urdf/my_robot.xacro (robot description, xacro)
@@ -22,5 +22,5 @@
       <origin xyz="0 0 0" rpy=" 0 0 0"/>
       <geometry>
-        <box size=".7 .4 .3"/>
+        <box size=".35 .2 .07"/>
       </geometry>
     </collision>
@@ -28,34 +28,34 @@
       <origin xyz="0 0 0" rpy=" 0 0 0"/>
       <geometry>
-        <box size=".7 .4 .3"/>
+        <box size=".35 .2 .07"/>
       </geometry>
     </visual>
     <collision name='back_caster_collision'>
-      <origin xyz="-0.15 0 -0.1" rpy=" 0 0 0"/>
+      <origin xyz="-0.15 0 -0.05" rpy=" 0 0 0"/>
       <geometry>
-        <sphere radius="0.1995"/>
+        <sphere radius="0.0298"/>
       </geometry>
     </collision>
     <visual name='back_caster_visual'>
-      <origin xyz="-0.15 0 -0.1" rpy=" 0 0 0"/>
+      <origin xyz="-0.15 0 -0.05" rpy=" 0 0 0"/>
       <geometry>
-        <sphere radius="0.205"/>
+        <sphere radius="0.0298"/>
       </geometry>
     </visual>
     <collision name='front_caster_collision'>
-      <origin xyz="0.15 0 -0.1" rpy=" 0 0 0"/>
+      <origin xyz="0.15 0 -0.05" rpy=" 0 0 0"/>
       <geometry>
-        <sphere radius="0.1995"/>
+        <sphere radius="0.0298"/>
       </geometry>
     </collision>
     <visual name='front_caster_visual'>
-      <origin xyz="0.15 0 -0.1" rpy=" 0 0 0"/>
+      <origin xyz="0.15 0 -0.05" rpy=" 0 0 0"/>
       <geometry>
-        <sphere radius="0.205"/>
+        <sphere radius="0.0298"/>
       </geometry>
     </visual>
   </link>
   <joint type="continuous" name="left_wheel_hinge">
-    <origin xyz="0 0.23 0" rpy="0 0 0"/>
+    <origin xyz="0 0.115 0" rpy="0 0 0"/>
     <child link="left_wheel"/>
     <parent link="chassis"/>
@@ -77,5 +77,5 @@
       <origin xyz="0 0 0" rpy="0 1.5707 1.5707"/>
       <geometry>
-        <cylinder length="0.05" radius="0.3"/>
+        <cylinder length="0.025" radius="0.08"/>
       </geometry>
     </visual>
@@ -83,10 +83,10 @@
       <origin xyz="0 0 0" rpy="0 1.5707 1.5707"/>
       <geometry>
-        <cylinder length="0.05" radius="0.3"/>
+        <cylinder length="0.025" radius="0.08"/>
       </geometry>
     </collision>
   </link>
   <joint type="continuous" name="right_wheel_hinge">
-    <origin xyz="0 -0.23 0" rpy="0 0 0"/>
+    <origin xyz="0 -0.115 0" rpy="0 0 0"/>
     <child link="right_wheel"/>
     <parent link="chassis"/>
@@ -108,5 +108,5 @@
       <origin xyz="0 0 0" rpy="0 1.5707 1.5707"/>
       <geometry>
-        <cylinder length="0.05" radius="0.3"/>
+        <cylinder length="0.025" radius="0.08"/>
       </geometry>
     </visual>
@@ -114,10 +114,10 @@
       <origin xyz="0 0 0" rpy="0 1.5707 1.5707"/>
       <geometry>
-        <cylinder length="0.05" radius="0.3"/>
+        <cylinder length="0.025" radius="0.08"/>
       </geometry>
     </collision>
   </link>
   <joint type="fixed" name="camera_joint">
-    <origin xyz="0.35 0 0.03" rpy="0 0 0"/>
+    <origin xyz="0.19 0 0" rpy="0 0 0"/>
     <child link="camera"/>
     <parent link="chassis"/>
@@ -149,5 +149,5 @@
   </link>
   <joint type="fixed" name="hokuyo_joint">
-    <origin xyz="0.3 0 0.18" rpy="0 0 0"/>
+    <origin xyz="0.15 0 0.07" rpy="0 0 0"/>
     <child link="hokuyo"/>
     <parent link="chassis"/>
